File: transection-vga/transection-vga.kicad_pcb (KiCad board)
At the start: 2 copper layers, 41.3 x 49.2 mm, 11 parts, among them J1 VGA_Socket, J2 Conn_01x15_Socket, J3 Conn_01x15_Socket, J4 VGA_Socket

Commit message: pcb edits
Other:
- board text added: "vga transectomy by aryl https://aryl.org"
Changed lines of the file:
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@@
+		)
+	)
+	(gr_text "vga transectomy by aryl\nhttps://aryl.org"
+		(at 135.75 86 -0)
+		(layer "F.SilkS")
+		(effects
+			(font
+				(size 0.8 0.8)
+				(thickness 0.1)
+			)
+			(justify bottom)
 		)
 	)
@@
 		)
 	)
+	(gr_text "vga transectomy by aryl\nhttps://aryl.org"
+		(at 135.75 111.25 0)
+		(layer "B.SilkS")
+		(effects
+			(font
+				(size 0.8 0.8)
+				(thickness 0.1)
+			)
+			(justify bottom mirror)
+		)
+	)

Commit message: pcb edits
Other:
- board text added: "vga transection by aryl https://aryl.org"
- board text removed: "vga transectomy by aryl https://aryl.org"
Changed lines of the file:
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@@
 		)
 	)
-	(gr_text "vga transectomy by aryl\nhttps://aryl.org"
-		(at 135.75 86 -0)
+	(gr_text "vga transection by aryl\nhttps://aryl.org"
+		(at 135.75 86 0)
 		(layer "F.SilkS")
 		(effects
@@
 		)
 	)
-	(gr_text "vga transectomy by aryl\nhttps://aryl.org"
+	(gr_text "vga transection by aryl\nhttps://aryl.org"
 		(at 135.75 111.25 0)
 		(layer "B.SilkS")
